Commit message: Fixing the robot position

File: sciclops_description/urdf/sciclops.urdf.xacro (robot description, xacro)
@@ -5,7 +5,7 @@
     <link name="${prefix}sciclops_base">
     <visual>
-      <origin xyz="0 0 0" rpy="0 0 0"/>
+      <origin xyz="0 0 0" rpy="1.5708 0 0"/>
       <geometry>
-        <mesh filename="package://sciclops_description/meshes/sciclops_base.STL" scale="0.001 0.001 0.001"/>
+        <mesh filename="package://sciclops_description/meshes/Sciclops_base.STL" scale="0.001 0.001 0.001"/>
       </geometry>
       <material name="black"/>
@@ -13,7 +13,7 @@
     <collision>
       <geometry>
-        <mesh filename="package://sciclops_description/meshes/sciclops_base.STL" scale="0.001 0.001 0.001"/>
+        <mesh filename="package://sciclops_description/meshes/Sciclops_base.STL" scale="0.001 0.001 0.001"/>
       </geometry>
-      <origin xyz="0 0 0" rpy="0 0 0"/>
+      <origin xyz="0 0 0" rpy="1.5708 0 0"/>
     </collision>
   </link>
@@ -22,11 +22,11 @@
       <origin xyz="0 0 0" rpy="0 0 0"/>
       <geometry>
-        <mesh filename="package://sciclops_description/meshes/sciclops_joint1.STL" scale="0.001 0.001 0.001"/>
+        <mesh filename="package://sciclops_description/meshes/Sciclops_joint1.STL" scale="0.001 0.001 0.001"/>
       </geometry>
-      <material name="aluminum"/>
+      <material name="white"/>
     </visual>
     <collision>
       <geometry>
-        <mesh filename="package://sciclops_description/meshes/sciclops_joint1.STL" scale="0.001 0.001 0.001"/>
+        <mesh filename="package://sciclops_description/meshes/Sciclops_joint1.STL" scale="0.001 0.001 0.001"/>
       </geometry>
       <origin xyz="0 0 0" rpy="0 0 0"/>
@@ -37,11 +37,11 @@
       <origin xyz="0 0 0" rpy="0 0 0"/>
       <geometry>
-        <mesh filename="package://sciclops_description/meshes/sciclops_joint2.STL" scale="0.001 0.001 0.001"/>
+        <mesh filename="package://sciclops_description/meshes/Sciclops_joint2.STL" scale="0.001 0.001 0.001"/>
       </geometry>
-      <material name="aluminum"/>
+      <material name="white"/>
     </visual>
     <collision>
       <geometry>
-        <mesh filename="package://sciclops_description/meshes/sciclops_joint2.STL" scale="0.001 0.001 0.001"/>
+        <mesh filename="package://sciclops_description/meshes/Sciclops_joint2.STL" scale="0.001 0.001 0.001"/>
       </geometry>
       <origin xyz="0 0 0" rpy="0 0 0"/>
@@ -52,11 +52,11 @@
       <origin xyz="0 0 0" rpy="0 0 0"/>
       <geometry>
-        <mesh filename="package://sciclops_description/meshes/sciclops_joint3.STL" scale="0.001 0.001 0.001"/>
+        <mesh filename="package://sciclops_description/meshes/Sciclops_joint3.STL" scale="0.001 0.001 0.001"/>
       </geometry>
-      <material name="aluminum"/>
+      <material name="white"/>
     </visual>
     <collision>
       <geometry>
-        <mesh filename="package://sciclops_description/meshes/sciclops_joint3.STL" scale="0.001 0.001 0.001"/>
+        <mesh filename="package://sciclops_description/meshes/Sciclops_joint3.STL" scale="0.001 0.001 0.001"/>
       </geometry>
       <origin xyz="0 0 0" rpy="0 0 0"/>
@@ -67,11 +67,11 @@
       <origin xyz="0 0 0" rpy="0 0 0"/>
       <geometry>
-        <mesh filename="package://sciclops_description/meshes/sciclops_joint4.STL" scale="0.001 0.001 0.001"/>
+        <mesh filename="package://sciclops_description/meshes/Sciclops_joint4.STL" scale="0.001 0.001 0.001"/>
       </geometry>
-      <material name="aluminum"/>
+      <material name="white"/>
     </visual>
     <collision>
       <geometry>
-        <mesh filename="package://sciclops_description/meshes/sciclops_joint4.STL" scale="0.001 0.001 0.001"/>
+        <mesh filename="package://sciclops_description/meshes/Sciclops_joint4.STL" scale="0.001 0.001 0.001"/>
       </geometry>
       <origin xyz="0 0 0" rpy="0 0 0"/>
@@ -79,17 +79,17 @@
   </link>
   <!-- Joints -->
-  <joint name="Sciclops_joint1" type="prismatic">
+  <joint name="Sciclops_joint1" type="revolute">
     <parent link="${prefix}sciclops_base"/>
     <child link="${prefix}sciclops_link1"/>
-    <axis xyz="0 0 1"/>
-    <origin xyz="0.055 -0.09 0.065" rpy="0 0 0"/>
-    <limit effort="1000.0" lower="0" upper="0.3" velocity="0.5"/>
+    <axis xyz="0 1 0"/>
+    <origin xyz="0 0 0" rpy="1.5708 0 0"/>
+    <limit effort="1000.0" lower="-3.1" upper="3.1" velocity="0.5"/>
   </joint>
   <joint name="Sciclops_joint2" type="prismatic">
     <parent link="${prefix}sciclops_link1"/>
     <child link="${prefix}sciclops_link2"/>
-    <axis xyz="0 0 1"/>
+    <axis xyz="0 1 0"/>
     <origin xyz="0 0 0" rpy="0 0 0"/>
-    <limit effort="1000.0" lower="0" upper="0.3" velocity="0.5"/>
+    <limit effort="1000.0" lower="-0.45" upper="0" velocity="0.5"/>
   </joint>
   <joint name="Sciclops_joint3" type="prismatic">
@@ -98,12 +98,12 @@
     <axis xyz="0 0 1"/>
     <origin xyz="0 0 0" rpy="0 0 0"/>
-    <limit effort="1000.0" lower="0" upper="0.3" velocity="0.5"/>
+    <limit effort="1000.0" lower="-0.1" upper="0" velocity="0.5"/>
   </joint>
-  <joint name="Sciclops_joint4" type="prismatic">
+  <joint name="Sciclops_joint4" type="revolute">
     <parent link="${prefix}sciclops_link3"/>
     <child link="${prefix}sciclops_link4"/>
-    <axis xyz="0 0 1"/>
+    <axis xyz="0 1 0"/>
     <origin xyz="0 0 0" rpy="0 0 0"/>
-    <limit effort="1000.0" lower="0" upper="0.3" velocity="0.5"/>
+    <limit effort="1000.0" lower="-3.1" upper="3.1" velocity="0.5"/>
   </joint>
   </xacro:macro>

File: sciclops_description/urdf/sciclops_robot.xacro (robot description, xacro)
@@ -13,5 +13,5 @@
     <child link="sciclops/sciclops_base"/>
     <axis xyz="0 0 0"/>
-    <origin xyz="0.2 -0.45 1.042" rpy="0 0 0"/>
+    <origin xyz="0.85 0.73 0.65" rpy="0 0 5.3"/>
     <limit effort="1000.0" lower="0" upper="0" velocity="0.5"/>
   </joint>

Commit message: Fixing the urdf

File: sciclops_description/urdf/sciclops.urdf.xacro (robot description, xacro)
@@ -84,5 +84,5 @@
     <axis xyz="0 1 0"/>
     <origin xyz="0 0 0" rpy="1.5708 0 0"/>
-    <limit effort="1000.0" lower="-3.1" upper="3.1" velocity="0.5"/>
+    <limit effort="1000.0" lower="-6.2" upper="6.2" velocity="0.5"/>
   </joint>
   <joint name="Sciclops_joint2" type="prismatic">
@@ -98,5 +98,5 @@
     <axis xyz="0 0 1"/>
     <origin xyz="0 0 0" rpy="0 0 0"/>
-    <limit effort="1000.0" lower="-0.1" upper="0" velocity="0.5"/>
+    <limit effort="1000.0" lower="-0.2" upper="0" velocity="0.5"/>
   </joint>
   <joint name="Sciclops_joint4" type="revolute">
@@ -104,6 +104,6 @@
     <child link="${prefix}sciclops_link4"/>
     <axis xyz="0 1 0"/>
-    <origin xyz="0 0 0" rpy="0 0 0"/>
-    <limit effort="1000.0" lower="-3.1" upper="3.1" velocity="0.5"/>
+    <origin xyz="-0.0001 0.611 -0.265" rpy="0 0 0"/>
+    <limit effort="1000.0" lower="-6.2" upper="6.2" velocity="0.5"/>
   </joint>
   </xacro:macro>

File: sciclops_description/urdf/sciclops_robot.xacro (robot description, xacro)
@@ -6,5 +6,5 @@
   <xacro:include filename="$(find sciclops_description)/urdf/module_carts.urdf.xacro" />
   <xacro:Module_Carts prefix="module_carts/"/>
-  <!-- Sealer -->
+  <!-- Sciclops -->
   <xacro:include filename="$(find sciclops_description)/urdf/sciclops.urdf.xacro" />
   <xacro:Sciclops prefix="sciclops/"/>
@@ -13,5 +13,5 @@
     <child link="sciclops/sciclops_base"/>
     <axis xyz="0 0 0"/>
-    <origin xyz="0.85 0.73 0.65" rpy="0 0 5.3"/>
+    <origin xyz="0 -0.04 1.05" rpy="0 0 5.1"/>
     <limit effort="1000.0" lower="0" upper="0" velocity="0.5"/>
   </joint>

Commit message: Creating a single urdf file

File: sciclops_description/urdf/sciclops.urdf.xacro (robot description, xacro)
@@ -3,5 +3,5 @@
   <!-- Links -->
   <xacro:macro name="Sciclops" params = "prefix">
-    <link name="${prefix}sciclops_base">
+  <link name="${prefix}sciclops_base">
     <visual>
       <origin xyz="0 0 0" rpy="1.5708 0 0"/>

Commit message: Adding gripper

File: sciclops_description/urdf/sciclops.urdf.xacro (robot description, xacro)
@@ -78,4 +78,34 @@
     </collision>
   </link>
+  <link name="${prefix}sciclops_link5">
+    <visual>
+      <origin xyz="0 0 0" rpy="0 0 0"/>
+      <geometry>
+        <mesh filename="package://sciclops_description/meshes/Sciclops_gripper_left.stl" scale="0.001 0.001 0.001"/>
+      </geometry>
+      <material name="white"/>
+    </visual>
+    <collision>
+      <geometry>
+        <mesh filename="package://sciclops_description/meshes/Sciclops_gripper_left.stl" scale="0.001 0.001 0.001"/>
+      </geometry>
+      <origin xyz="0 0 0" rpy="0 0 0"/>
+    </collision>
+  </link>
+  <link name="${prefix}sciclops_link6">
+    <visual>
+      <origin xyz="0 0 0" rpy="0 0 0"/>
+      <geometry>
+        <mesh filename="package://sciclops_description/meshes/Sciclops_gripper_right.stl" scale="0.001 0.001 0.001"/>
+      </geometry>
+      <material name="white"/>
+    </visual>
+    <collision>
+      <geometry>
+        <mesh filename="package://sciclops_description/meshes/Sciclops_gripper_right.stl" scale="0.001 0.001 0.001"/>
+      </geometry>
+      <origin xyz="0 0 0" rpy="0 0 0"/>
+    </collision>
+  </link>
   <!-- Joints -->
   <joint name="Sciclops_joint1" type="revolute">
@@ -107,4 +137,19 @@
     <limit effort="1000.0" lower="-6.2" upper="6.2" velocity="0.5"/>
   </joint>
+  <joint name="Sciclops_gripper" type="prismatic">
+    <parent link="${prefix}sciclops_link4"/>
+    <child link="${prefix}sciclops_link5"/>
+    <axis xyz="-1 0 0"/>
+    <origin xyz="-0.00 0 0.0012" rpy="0 0 0"/>
+    <limit effort="1000.0" lower="0.0" upper="0.01" velocity="0.5"/>
+  </joint>
+  <joint name="Sciclops_gripper_mirror" type="prismatic">
+    <parent link="${prefix}sciclops_link4"/>
+    <child link="${prefix}sciclops_link6"/>
+    <axis xyz="1 0 0"/>
+    <origin xyz="0.00 0 -0.0012" rpy="0 0 0"/>
+    <limit effort="1000.0" lower="0.0" upper="0.01" velocity="0.5"/>
+    <mimic joint="Sciclops_gripper" multiplier="1"/>
+  </joint>
   </xacro:macro>
 </robot>
